File: Charger Shutdown Circuit.kicad_sch (KiCad schematic)
At the start: 25 parts, among them J1 Charger Shutdown Button conne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, J2 Conn_01x02_Pin, J3 Conn_01x02_Pin, J4 Conn_01x02_Pin, J5 Conn_01x04_Pin, K1 G5Q-1, Q1 PMOS IRF5305, Q2 PMOS IRF5305, Q4 BJT, Q5 BJT

Commit message: Added Status LED and organized schematic
Parts:
- added D3: LED, symbol Device:LED
- added R14: 10k, Resistor_THT:R_Axial_DIN0309_L9.0mm_D3.2mm_P15.24mm_Horizontal, symbol Device:R
Connections:
- net GND: now also D3.1 (K)
- net Relayoutput: now also R14.2
- new net: D3.2 (A), R14.1
Other:
- note added: "IO Lines"
- note added: "Main Circuit"
- note added: "Status LED"
- moved on the sheet: C1, D1, D2, J1, J2, J3, J4, J5, JP1, JP2, JP3, K1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

Commit message: Minor changes
Parts:
- renumbered J3 to J1, J5 to J2, J4 to J3, J2 to J4, J1 to J5, Q4 to Q1, Q1 to Q2, Q5 to Q3, Q2 to Q4, R8 to R1, R14 to R10, R11 to R2, R1 to R3, R5 to R4, R9 to R5, R12 to R6, R2 to R7, R6 to R8, R4 to R9
Changed lines of the file:
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@@
 	)
 	(junction
-		(at 40.64 102.87)
-		(diameter 0)
-		(color 0 0 0 0)
-	)
-	(junction
 		(at 153.67 127)
 		(diameter 0)
@@
 	(wire
 		(pts
-			(xy 35.56 102.87) (xy 40.64 102.87)
-		)
-		(stroke
-			(width 0)
-			(type default)
-		)
-	)
-	(wire
-		(pts
-			(xy 40.64 97.79) (xy 40.64 102.87)
-		)
-		(stroke
-			(width 0)
-			(type default)
-		)
-	)
-	(wire
-		(pts
 			(xy 97.79 113.03) (xy 97.79 110.49)
 		)
@@
 	(wire
 		(pts
-			(xy 40.64 102.87) (xy 57.15 102.87)
+			(xy 35.56 102.87) (xy 57.15 102.87)
 		)
 		(stroke
@@
 		)
 	)
-	(label "LV_Status"
-		(at 40.64 97.79 0)
-		(effects
-			(font
-				(size 1.27 1.27)
-			)
-			(justify left bottom)
-		)
-	)
 	(label "Relayoutput"
 		(at 198.12 39.37 180)
@@
 		(in_pos_files yes)
 		(dnp no)
-		(property "Reference" "R5"
+		(property "Reference" "R4"
 			(at 58.8772 116.9416 0)
 			(show_name no)
@@
 			(project "Charger Shutdown Circuit"
 				(path "/301bc50e-ce57-49bf-a5a2-8423cd4c9567"
-					(reference "R5")
+					(reference "R4")
 					(unit 1)
 				)
@@
 		(in_pos_files yes)
 		(dnp no)
-		(property "Reference" "R12"
+		(property "Reference" "R6"
 			(at 79.1972 130.9116 0)
 			(show_name no)
@@
 			(project "Charger Shutdown Circuit"
 				(path "/301bc50e-ce57-49bf-a5a2-8423cd4c9567"
-					(reference "R12")
+					(reference "R6")
 					(unit 1)
 				)
@@
 		(in_pos_files yes)
 		(dnp no)
-		(property "Reference" "R4"
+		(property "Reference" "R9"
 			(at 149.0472 110.5916 0)
 			(show_name no)
@@
 			(project "Charger Shutdown Circuit"
 				(path "/301bc50e-ce57-49bf-a5a2-8423cd4c9567"
-					(reference "R4")
+					(reference "R9")
 					(unit 1)
 				)
@@
 		(dnp no)
 		(fields_autoplaced yes)
-		(property "Reference" "#PWR01"
+		(property "Reference" "#PWR04"
 			(at 73.66 54.61 0)
 			(hide yes)
@@
 			(project "Charger Shutdown Circuit"
 				(path "/301bc50e-ce57-49bf-a5a2-8423cd4c9567"
-					(reference "#PWR01")
+					(reference "#PWR04")
 					(unit 1)
 				)
@@
 		(dnp no)
 		(fields_autoplaced yes)
-		(property "Reference" "J3"
+		(property "Reference" "J1"
 			(at 24.765 27.94 0)
 			(show_name no)
@@
 			(project "Charger Shutdown Circuit"
 				(path "/301bc50e-ce57-49bf-a5a2-8423cd4c9567"
-					(reference "J3")
+					(reference "J1")
 					(unit 1)
 				)
@@
 		(dnp no)
 		(fields_autoplaced yes)
-		(property "Reference" "#PWR08"
+		(property "Reference" "#PWR010"
 			(at 226.06 52.07 0)
 			(hide yes)
@@
 			(project "Charger Shutdown Circuit"
 				(path "/301bc50e-ce57-49bf-a5a2-8423cd4c9567"
-					(reference "#PWR08")
+					(reference "#PWR010")
 					(unit 1)
 				)
@@
 		(in_pos_files yes)
 		(dnp no)
-		(property "Reference" "#PWR09"
+		(property "Reference" "#PWR02"
 			(at 45.72 143.51 0)
 			(hide yes)
@@
 			(project "Charger Shutdown Circuit"
 				(path "/301bc50e-ce57-49bf-a5a2-8423cd4c9567"
-					(reference "#PWR09")
+					(reference "#PWR02")
 					(unit 1)
 				)
@@
 		(in_pos_files yes)
 		(dnp no)
-		(property "Reference" "#PWR010"
+		(property "Reference" "#PWR05"
 			(at 77.47 143.51 0)
 			(hide yes)
@@
 			(project "Charger Shutdown Circuit"
 				(path "/301bc50e-ce57-49bf-a5a2-8423cd4c9567"
-					(reference "#PWR010")
+					(reference "#PWR05")
 					(unit 1)
 				)
@@
 		(dnp no)
 		(fields_autoplaced yes)
-		(property "Reference" "#PWR03"
+		(property "Reference" "#PWR08"
 			(at 171.45 121.92 0)
 			(hide yes)
@@
 			(project "Charger Shutdown Circuit"
 				(path "/301bc50e-ce57-49bf-a5a2-8423cd4c9567"
-					(reference "#PWR03")
+					(reference "#PWR08")
 					(unit 1)
 				)
@@
 		(in_pos_files yes)
 		(dnp no)
-		(property "Reference" "Q4"
+		(property "Reference" "Q1"
 			(at 59.436 127.1016 0)
 			(show_name no)
@@
 			(project "Charger Shutdown Circuit"
 				(path "/301bc50e-ce57-49bf-a5a2-8423cd4c9567"
-					(reference "Q4")
+					(reference "Q1")
 					(unit 1)
 				)
@@
 		(in_pos_files yes)
 		(dnp no)
-		(property "Reference" "R8"
+		(property "Reference" "R1"
 			(at 41.8084 129.9972 0)
 			(show_name no)
@@
 			(project "Charger Shutdown Circuit"
 				(path "/301bc50e-ce57-49bf-a5a2-8423cd4c9567"
-					(reference "R8")
+					(reference "R1")
 					(unit 1)
 				)
@@
 		(in_pos_files yes)
 		(dnp no)
-		(property "Reference" "#PWR02"
+		(property "Reference" "#PWR01"
 			(at 35.56 118.11 0)
 			(hide yes)
@@
 			(project "Charger Shutdown Circuit"
 				(path "/301bc50e-ce57-49bf-a5a2-8423cd4c9567"
-					(reference "#PWR02")
+					(reference "#PWR01")
 					(unit 1)
 				)
@@
 		(in_pos_files yes)
 		(dnp no)
-		(property "Reference" "#PWR06"
+		(property "Reference" "#PWR03"
 			(at 57.15 140.97 0)
 			(hide yes)
@@
 			(project "Charger Shutdown Circuit"
 				(path "/301bc50e-ce57-49bf-a5a2-8423cd4c9567"
-					(reference "#PWR06")
+					(reference "#PWR03")
 					(unit 1)
 				)
@@
 		(in_pos_files yes)
 		(dnp no)
-		(property "Reference" "#PWR07"
+		(property "Reference" "#PWR06"
 			(at 88.9 140.97 0)
 			(hide yes)
@@
 			(project "Charger Shutdown Circuit"
 				(path "/301bc50e-ce57-49bf-a5a2-8423cd4c9567"
-					(reference "#PWR07")
+					(reference "#PWR06")
 					(unit 1)
 				)
@@
 		(dnp no)
 		(fields_autoplaced yes)
-		(property "Reference" "J5"
+		(property "Reference" "J2"
 			(at 24.765 41.91 0)
 			(show_name no)
@@
 			(project "Charger Shutdown Circuit"
 				(path "/301bc50e-ce57-49bf-a5a2-8423cd4c9567"
-					(reference "J5")
+					(reference "J2")
 					(unit 1)
 				)
@@
 		(dnp no)
 		(fields_autoplaced yes)
-		(property "Reference" "#PWR05"
+		(property "Reference" "#PWR09"
 			(at 171.45 133.35 0)
 			(hide yes)
@@
 			(project "Charger Shutdown Circuit"
 				(path "/301bc50e-ce57-49bf-a5a2-8423cd4c9567"
-					(reference "#PWR05")
+					(reference "#PWR09")
 					(unit 1)
 				)
@@
 		(in_pos_files yes)
 		(dnp no)
-		(property "Reference" "R6"
+		(property "Reference" "R8"
 			(at 90.6272 116.9416 0)
 			(show_name no)
@@
 			(project "Charger Shutdown Circuit"
 				(path "/301bc50e-ce57-49bf-a5a2-8423cd4c9567"
-					(reference "R6")
+					(reference "R8")
 					(unit 1)
 				)
@@
 		(dnp no)
 		(fields_autoplaced yes)
-		(property "Reference" "J4"
+		(property "Reference" "J3"
 			(at 65.405 27.94 0)
 			(show_name no)
@@
 			(project "Charger Shutdown Circuit"
 				(path "/301bc50e-ce57-49bf-a5a2-8423cd4c9567"
-					(reference "J4")
+					(reference "J3")
 					(unit 1)
 				)
@@
 		(in_pos_files yes)
 		(dnp no)
-		(property "Reference" "Q5"
+		(property "Reference" "Q3"
 			(at 91.186 127.1016 0)
 			(show_name no)
@@
 			(project "Charger Shutdown Circuit"
 				(path "/301bc50e-ce57-49bf-a5a2-8423cd4c9567"
-					(reference "Q5")
+					(reference "Q3")
 					(unit 1)
 				)
@@
 		(in_pos_files yes)
 		(dnp no)
-		(property "Reference" "#PWR04"
+		(property "Reference" "#PWR07"
 			(at 147.32 125.73 0)
 			(hide yes)
@@
 			(project "Charger Shutdown Circuit"
 				(path "/301bc50e-ce57-49bf-a5a2-8423cd4c9567"
-					(reference "#PWR04")
+					(reference "#PWR07")
 					(unit 1)
 				)
@@
 		(in_pos_files yes)
 		(dnp no)
-		(property "Reference" "J1"
+		(property "Reference" "J5"
 			(at 123.952 40.894 0)
 			(show_name no)
@@
 			(project "Charger Shutdown Circuit"
 				(path "/301bc50e-ce57-49bf-a5a2-8423cd4c9567"
-					(reference "J1")
+					(reference "J5")
 					(unit 1)
 				)
@@
 		(in_pos_files yes)
 		(dnp no)
-		(property "Reference" "R2"
+		(property "Reference" "R7"
 			(at 90.6272 106.7816 0)
 			(show_name no)
@@
 			(project "Charger Shutdown Circuit"
 				(path "/301bc50e-ce57-49bf-a5a2-8423cd4c9567"
-					(reference "R2")
+					(reference "R7")
 					(unit 1)
 				)
@@
 		(in_pos_files yes)
 		(dnp no)
-		(property "Reference" "R9"
+		(property "Reference" "R5"
 			(at 73.5584 129.9972 0)
 			(show_name no)
@@
 			(project "Charger Shutdown Circuit"
 				(path "/301bc50e-ce57-49bf-a5a2-8423cd4c9567"
-					(reference "R9")
+					(reference "R5")
 					(unit 1)
 				)
@@
 		(dnp no)
 		(fields_autoplaced yes)
-		(property "Reference" "R14"
+		(property "Reference" "R10"
 			(at 205.74 33.02 90)
 			(show_name no)
@@
 			(project "Charger Shutdown Circuit"
 				(path "/301bc50e-ce57-49bf-a5a2-8423cd4c9567"
-					(reference "R14")
+					(reference "R10")
 					(unit 1)
 				)
@@
 		(in_pos_files yes)
 		(dnp no)
-		(property "Reference" "Q1"
+		(property "Reference" "Q2"
 			(at 66.04 96.7232 90)
 			(show_name no)
@@
 			(project "Charger Shutdown Circuit"
 				(path "/301bc50e-ce57-49bf-a5a2-8423cd4c9567"
-					(reference "Q1")
+					(reference "Q2")
 					(unit 1)
 				)
@@
 		(in_pos_files yes)
 		(dnp no)
-		(property "Reference" "Q2"
+		(property "Reference" "Q4"
 			(at 97.79 96.7232 90)
 			(show_name no)
@@
 			(project "Charger Shutdown Circuit"
 				(path "/301bc50e-ce57-49bf-a5a2-8423cd4c9567"
-					(reference "Q2")
+					(reference "Q4")
 					(unit 1)
 				)
@@
 		(in_pos_files yes)
 		(dnp no)
-		(property "Reference" "R1"
+		(property "Reference" "R3"
 			(at 58.8772 106.7816 0)
 			(show_name no)
@@
 			(project "Charger Shutdown Circuit"
 				(path "/301bc50e-ce57-49bf-a5a2-8423cd4c9567"
-					(reference "R1")
+					(reference "R3")
 					(unit 1)
 				)
@@
 		(in_pos_files yes)
 		(dnp no)
-		(property "Reference" "R11"
+		(property "Reference" "R2"
 			(at 47.4472 130.9116 0)
 			(show_name no)
@@
 			(project "Charger Shutdown Circuit"
 				(path "/301bc50e-ce57-49bf-a5a2-8423cd4c9567"
-					(reference "R11")
+					(reference "R2")
 					(unit 1)
 				)
@@
 		(dnp no)
 		(fields_autoplaced yes)
-		(property "Reference" "J2"
+		(property "Reference" "J4"
 			(at 116.205 27.94 0)
 			(show_name no)
@@
 			(project "Charger Shutdown Circuit"
 				(path "/301bc50e-ce57-49bf-a5a2-8423cd4c9567"
-					(reference "J2")
+					(reference "J4")
 					(unit 1)
 				)
